File: circuit/encoder_disk/encoder_disk.kicad_pcb (KiCad board)
At the start: 2 copper layers, 21 x 21 mm, 7 parts, among them J1 Conn_01x04

Commit message: 整理
Parts:
- removed C1: 0.1u, Capacitor_SMD:C_0603_1608Metric_Pad1.08x0.95mm_HandSolder
- removed J1: Conn_01x04, Connector_PinHeader_2.54mm:PinHeader_1x04_P2.54mm_Vertical
- removed R1: 220, Resistor_SMD:R_0603_1608Metric_Pad0.98x0.95mm_HandSolder
- removed R2, R3: 1k, Resistor_SMD:R_0603_1608Metric_Pad0.98x0.95mm_HandSolder
- removed U1: ~, mylib:NJL5820R
