File: circuit/encoder_circuit/encoder_circuit.kicad_pcb (KiCad board)
At the start: 2 copper layers, 2.5 x 2.6 mm, 6 parts, among them J1 Conn_01x04

Commit message: step
Parts:
- added G***: LOGO, Symbol:sh_10mm, F.Cu at (141.8, 92.2)
- added REF**: MountingHole_2.2mm_M2, MountingHole:MountingHole_2.2mm_M2, F.Cu at (131.8, 101.0)
- added REF**: MountingHole_2.2mm_M2, MountingHole:MountingHole_2.2mm_M2, F.Cu at (151.8, 101.0)
- C1, R1, R2, R3, U1: moved to B.Cu
- moved J1 13.9 mm to (137.9, 101.0), turned to 90 degrees
- moved U1 8.81 mm to (141.8, 86.0), turned to 180 degrees
- moved R2 8.79 mm to (139.2, 97.2)
- moved R1 8.39 mm to (144.2, 97.2), turned to 180 degrees
- moved C1 7.23 mm to (144.2, 93.5), turned to 180 degrees
- moved R3 6.71 mm to (139.2, 93.5)
Routing:
- net +3.3V: track 0.00 -> 35.1 mm
- net Net-(J1-Pin_2): track 0.00 -> 17.2 mm
- net GND: track 0.00 -> 16.6 mm, vias 0 -> 11
- net Net-(J1-Pin_3): track 0.00 -> 15.6 mm
- net Net-(U1-Anode): track 0.00 -> 13.1 mm
- added copper zone on B.Cu, net GND
- added copper zone on F.Cu, net GND
Other:
- board size 2.5 x 2.6 mm -> 27 x 23 mm

Commit message: エンコーダ基板の回路図更新
Parts:
- J1: footprint Connector_PinHeader_2.54mm:PinHeader_1x04_P2.54mm_Vertical -> Connector_JST:JST_PH_B4B-PH-K_1x04_P2.00mm_Vertical
- moved J1 1.28 mm to (139.1, 100.5), turned to 0 degrees
- turned U1 to -90 degrees
Routing:
- net +3.3V: track 35.1 -> 23.6 mm
- net GND: track 16.6 -> 11.4 mm
- net Net-(J1-Pin_2): track 17.2 -> 14.2 mm
- net Net-(J1-Pin_3): track 15.6 -> 13.1 mm
- net Net-(U1-Anode): track 13.1 -> 10.9 mm

Commit message: エンコーダ基板修正
Parts:
- removed R2, R3: 1k, Resistor_SMD:R_0603_1608Metric_Pad0.98x0.95mm_HandSolder
- removed the REF** at (131.8, 101.0)
- removed the REF** at (151.8, 101.0)
- added REF**: MountingHole_2.2mm_M2, MountingHole:MountingHole_2.2mm_M2, F.Cu at (121.6, 90.0)
- added REF**: MountingHole_2.2mm_M2, MountingHole:MountingHole_2.2mm_M2, F.Cu at (138.4, 90.0)
- moved C1 19.4 mm to (130.0, 80.3), turned to 0 degrees
- moved R1 18.1 mm to (127.0, 91.6), turned to 90 degrees
- moved U1 12.3 mm to (130.0, 82.5)
- moved G*** 12.0 mm to (130.0, 90.0)
- moved J1 6.94 mm to (133.0, 97.2), turned to 180 degrees
Connections:
- J1 pad 1: +3.3V -> GND
- J1 pad 4: GND -> +3.3V
- U1 pad 3: Net-(J1-Pin_3) -> Net-(J1-Pin_2)
- U1 pad 4: Net-(J1-Pin_2) -> Net-(J1-Pin_3)
Routing:
- net GND: track 11.4 -> 2.22 mm, vias 11 -> 25
- net +3.3V: track 23.6 -> 22.1 mm
- net Net-(U1-Anode): track 10.9 -> 10.1 mm
- net Net-(J1-Pin_3): track 13.1 -> 13.8 mm
Other:
- board size 27 x 23 mm -> 22 x 22 mm
